Commit message: update inertia

File: Arm/URDF/right_arm/src/hopejr_arm_description/urdf/hopejr_arm.urdf (robot description, URDF)
Before this commit: robot hopejr_arm, 7 links, 6 joints
Links:
- link base_link: mass 2.0 -> 1.260139
- link forearm: mass 2.0 -> 0.208355
- link lower_elbow: mass 2.0 -> 0.1882
- link shoulder_roll: mass 2.0 -> 0.422614
- link shoulder_yaw: mass 2.0 -> 0.252213
- link upper_elbow: mass 2.0 -> 0.243803

File: Arm/URDF/right_arm/src/hopejr_arm_description/urdf/hopejr_arm.urdf.xacro (robot description, xacro)
@@ -17,6 +17,6 @@
             <inertial>
                 <origin xyz="-0.02 0 0.028" rpy="0 0 0"/>
-                <mass value="2.0"/>
-                <inertia ixx="0.000213" ixy="0" ixz="0" iyy="0.007034" iyz="0" izz="0.008104"/>
+                <mass value="1.260139"/>
+                <inertia ixx="0.003444" ixy="0.000000060725" ixz="0.000000223974" iyy="0.003173" iyz="0.0003306" izz="0.002316"/>
             </inertial>
         </link>
@@ -41,6 +41,6 @@
             <inertial>
                 <origin xyz="0 0 0" rpy="0 0 0"/>
-                <mass value="2.0"/>
-                <inertia ixx="0.01" ixy="0" ixz="0" iyy="0.01" iyz="0" izz="0.01"/>
+                <mass value="0.252213"/>
+                <inertia ixx="0.0001227" ixy="0.000000629536" ixz="-0.000000333468" iyy="0.0001678" iyz="-0.000000674054" izz="0.0001553"/>
             </inertial>
         </link>
@@ -67,6 +67,6 @@
             <inertial>
                 <origin xyz="-0.02 0 0.028" rpy="0 0 0"/>
-                <mass value="2.0"/>
-                <inertia ixx="0.01" ixy="0" ixz="0" iyy="0.01" iyz="0" izz="0.01"/>
+                <mass value="0.422614"/>
+                <inertia ixx="0.0006959" ixy="0.000006134701" ixz="-0.000083430347" iyy="0.0007655" iyz="0.000025066263" izz="0.0002446"/>
             </inertial>
         </link>
@@ -92,6 +92,6 @@
             <inertial>
                 <origin xyz="-0.02 0 0.028" rpy="0 0 0"/>
-                <mass value="2.0"/>
-                <inertia ixx="0.01" ixy="0" ixz="0" iyy="0.01" iyz="0" izz="0.01"/>
+                <mass value="0.243803"/>
+                <inertia ixx="0.0003227" ixy="-0.000000062111" ixz="-0.0001214" iyy="0.0003959" iyz="-0.000000048168" izz="0.0001746"/>
             </inertial>
         </link>
@@ -117,6 +117,6 @@
             <inertial>
                 <origin xyz="-0.02 0 0.028" rpy="0 0 0"/>
-                <mass value="2.0"/>
-                <inertia ixx="0.01" ixy="0" ixz="0" iyy="0.01" iyz="0" izz="0.01"/>
+                <mass value="0.1882"/>
+                <inertia ixx="0.0001196" ixy="0.000002288885" ixz="0.000001137302" iyy="0.000096307138" iyz="0.000003223544" izz="0.0001047"/>
             </inertial>
         </link>
@@ -143,6 +143,6 @@
             <inertial>
                 <origin xyz="-0.02 0 0.028" rpy="0 0 0"/>
-                <mass value="2.0"/>
-                <inertia ixx="0.01" ixy="0" ixz="0" iyy="0.01" iyz="0" izz="0.01"/>
+                <mass value="0.208355"/>
+                <inertia ixx="0.0002051" ixy="0.000000044894" ixz="-0.000004226706" iyy="0.0002222" iyz="-0.000002431512" izz="0.0001122"/>
             </inertial>
         </link>
