Commit message: update inertia

File: Arm/URDF/right_arm/src/hopejr_right_arm_description/urdf/hopejr_right_arm.urdf (robot description, URDF)
Before this commit: robot hopejr_right_arm_robot, 52 links, 51 joints
Links:
- link base_link: mass 2.0 -> 1.260139
- link forearm: mass 2.0 -> 0.208355
- link hand_base_link: mass 2.0 -> 0.03323
- link hand_hand: mass 2.0 -> 0.252893
- link hand_index_dip_1: mass 2.0 -> 0.005093
- link hand_index_dip_2: mass 2.0 -> 0.005429
- link hand_index_mcp_1: mass 2.0 -> 0.004836
- link hand_index_mcp_2: mass 2.0 -> 0.001654
- link hand_index_pip: mass 2.0 -> 0.005708
- link hand_middle_dip_1: mass 2.0 -> 0.005093
- link hand_middle_dip_2: mass 2.0 -> 0.005429
- link hand_middle_mcp_1: mass 2.0 -> 0.004836
- link hand_middle_mcp_2: mass 2.0 -> 0.001654
- link hand_middle_pip: mass 2.0 -> 0.005708
- link hand_pinky_dip_1: mass 2.0 -> 0.005093
- link hand_pinky_dip_2: mass 2.0 -> 0.005429
- link hand_pinky_mcp_1: mass 2.0 -> 0.004836
- link hand_pinky_mcp_2: mass 2.0 -> 0.001654
- link hand_pinky_pip: mass 2.0 -> 0.005708
- link hand_ring_dip_1: mass 2.0 -> 0.005093
- link hand_ring_dip_2: mass 2.0 -> 0.005429
- link hand_ring_mcp_1: mass 2.0 -> 0.004836
- link hand_ring_mcp_2: mass 2.0 -> 0.001654
- link hand_ring_pip: mass 2.0 -> 0.005708
- link hand_thumb_dip: mass 2.0 -> 0.005429
- link hand_thumb_mcp_2: mass 2.0 -> 0.008776
- link hand_thumb_pip_1: mass 2.0 -> 0.007142
- link hand_thumb_pip_2: mass 2.0 -> 0.006089
- link lower_elbow: mass 2.0 -> 0.1882
- link shoulder_roll: mass 2.0 -> 0.422614
- link shoulder_yaw: mass 2.0 -> 0.252213
- link upper_elbow: mass 2.0 -> 0.243803

Commit message: update mass of supports

File: Arm/URDF/right_arm/src/hopejr_right_arm_description/urdf/hopejr_right_arm.urdf (robot description, URDF)
Before this commit: robot hopejr_right_arm_robot, 52 links, 51 joints
Links:
- link hand_index_dip_1_support: mass 2.0 -> 0.0000000000001
- link hand_index_dip_2_support: mass 2.0 -> 0.0000000000001
- link hand_index_mcp_2_support: mass 2.0 -> 0.0000000000001
- link hand_index_pip_support: mass 2.0 -> 0.0000000000001
- link hand_middle_dip_1_support: mass 2.0 -> 0.0000000000001
- link hand_middle_dip_2_support: mass 2.0 -> 0.0000000000001
- link hand_middle_mcp_2_support: mass 2.0 -> 0.0000000000001
- link hand_middle_pip_support: mass 2.0 -> 0.0000000000001
- link hand_pinky_dip_1_support: mass 2.0 -> 0.0000000000001
- link hand_pinky_dip_2_support: mass 2.0 -> 0.0000000000001
- link hand_pinky_mcp_2_support: mass 2.0 -> 0.0000000000001
- link hand_pinky_pip_support: mass 2.0 -> 0.0000000000001
- link hand_ring_dip_1_support: mass 2.0 -> 0.0000000000001
- link hand_ring_dip_2_support: mass 2.0 -> 0.0000000000001
- link hand_ring_mcp_2_support: mass 2.0 -> 0.0000000000001
- link hand_ring_pip_support: mass 2.0 -> 0.0000000000001
- link hand_thumb_dip_support: mass 2.0 -> 0.0000000000001
- link hand_thumb_pip_1_support: mass 2.0 -> 0.0000000000001
- link hand_thumb_pip_2_support: mass 2.0 -> 0.0000000000001
